Commit message: rtab

File: leo_rover/urdf/leo_with_lidar.urdf (robot description, URDF)
Before this commit: robot leo_erc_sim, 22 links, 21 joints
Links:
- added link lidar, mass 1e-05; collision cylinder length=0.08 radius=0.06; visual cylinder length=0.08 radius=0.06
Joints:
- added joint lidar_joint: type fixed, parent rocker_L_link, child lidar, origin xyz=0.2 0 0.17 rpy=0 0 2.792527, axis 0 1 0
