Commit message: Navigation with lidar added

File: leo_rover/urdf/leo_erc_sim.urdf (robot description, URDF)
Before this commit: robot leo_erc_sim, 22 links, 21 joints
Links:
- added link lidar, mass 1e-05; collision cylinder length=0.08 radius=0.06; visual cylinder length=0.08 radius=0.06
Joints:
- added joint lidar_joint: type fixed, parent rocker_L_link, child lidar, origin xyz=0.2 0 0.17 rpy=0 0 0, axis 0 1 0

File: leo_rover/urdf/rover.urdf (robot description, URDF)
Before this commit: robot rover, 12 links, 11 joints
Links:
- removed link chassis
- added link base_footprint
- added link base_link, mass 7; collision box size=0.55 0.5 0.2; visual box size=0.55 0.5 0.2
Joints:
- added joint base_footprint_joint: type fixed, parent base_link, child base_footprint, origin xyz=0 0 0 rpy=0 0 0
- joint camera_joint: parent chassis -> base_link
- joint gps_joint: parent chassis -> base_link
- joint imu_joint: parent chassis -> base_link
- joint left_wheel_hinge_back: parent chassis -> base_link
- joint left_wheel_hinge_front: parent chassis -> base_link
- joint lidar_joint: parent chassis -> base_link
- joint right_wheel_hinge_back: parent chassis -> base_link
- joint right_wheel_hinge_front: parent chassis -> base_link
- joint robot_footprint_joint: child chassis -> base_link
- joint zed2_joint: parent chassis -> base_link

Commit message: tuning

File: leo_rover/urdf/leo_erc_sim.urdf (robot description, URDF)
Before this commit: robot leo_erc_sim, 23 links, 22 joints
Joints:
- joint lidar_joint: origin xyz=0.2 0 0.17 rpy=0 0 0 -> xyz=0.2 0 0.17 rpy=0 0 2.792527

Commit message: goal setter

File: leo_rover/urdf/leo_erc_sim.urdf (robot description, URDF)
Before this commit: robot leo_erc_sim, 22 links, 21 joints
Links:
- link base_link: geometry collision mesh filename=/home/akshat/ros2_ws/src/leo_rover/models/Chassis_outline.s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; visual mesh filename=/home/akshat/ros2_ws/src/leo_rover/models/Chassis.dae
- link erc_payload_link: geometry collision mesh filename=/home/akshat/ros2_ws/src/leo_rover/models/ERC2021payload_ou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; visual mesh filename=/home/akshat/ros2_ws/src/leo_rover/models/ERC2021payload.dae
- link rocker_L_link: geometry collision mesh filename=/home/akshat/ros2_ws/src/leo_rover/models/Rocker_outline.stl; visual mesh filename=/home/akshat/ros2_ws/src/leo_rover/models/Rocker.dae
- link rocker_R_link: geometry collision mesh filename=/home/akshat/ros2_ws/src/leo_rover/models/Rocker_outline.stl; visual mesh filename=/home/akshat/ros2_ws/src/leo_rover/models/Rocker.dae
- link wheel_FL_link: geometry collision cylinder length=0.04 radius=0.0625; collision cylinder length=0.07 radius=0.057
- link wheel_FR_link: geometry collision cylinder length=0.04 radius=0.0625; collision cylinder length=0.07 radius=0.057
- link wheel_RL_link: geometry collision cylinder length=0.04 radius=0.0625; collision cylinder length=0.07 radius=0.057
- link wheel_RR_link: geometry collision cylinder length=0.04 radius=0.0625; collision cylinder length=0.07 radius=0.057
- link zed2_camera_center: geometry collision mesh filename=/home/akshat/ros2_ws/src/leo_rover/models/ZED2.dae; visual mesh filename=/home/akshat/ros2_ws/src/leo_rover/models/ZED2.dae
- link zed2_tilt_head_link: geometry collision mesh filename=/home/akshat/ros2_ws/src/leo_rover/models/Manfrotto_head.dae; visual mesh filename=/home/akshat/ros2_ws/src/leo_rover/models/Manfrotto_head.dae

File: leo_rover/urdf/leo_with_lidar.urdf (robot description, URDF)
Before this commit: robot leo_erc_sim, 23 links, 22 joints
Links:
- link base_link: geometry collision mesh filename=/home/akshat/ros2_ws/src/leo_rover/models/Chassis_outline.s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; visual mesh filename=/home/akshat/ros2_ws/src/leo_rover/models/Chassis.dae
- link erc_payload_link: geometry collision mesh filename=/home/akshat/ros2_ws/src/leo_rover/models/ERC2021payload_ou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; visual mesh filename=/home/akshat/ros2_ws/src/leo_rover/models/ERC2021payload.dae
- link rocker_L_link: geometry collision mesh filename=/home/akshat/ros2_ws/src/leo_rover/models/Rocker_outline.stl; visual mesh filename=/home/akshat/ros2_ws/src/leo_rover/models/Rocker.dae
- link rocker_R_link: geometry collision mesh filename=/home/akshat/ros2_ws/src/leo_rover/models/Rocker_outline.stl; visual mesh filename=/home/akshat/ros2_ws/src/leo_rover/models/Rocker.dae
- link wheel_FL_link: geometry collision cylinder length=0.04 radius=0.0625; collision cylinder length=0.07 radius=0.057
- link wheel_FR_link: geometry collision cylinder length=0.04 radius=0.0625; collision cylinder length=0.07 radius=0.057
- link wheel_RL_link: geometry collision cylinder length=0.04 radius=0.0625; collision cylinder length=0.07 radius=0.057
- link wheel_RR_link: geometry collision cylinder length=0.04 radius=0.0625; collision cylinder length=0.07 radius=0.057
- link zed2_camera_center: geometry collision mesh filename=/home/akshat/ros2_ws/src/leo_rover/models/ZED2.dae; visual mesh filename=/home/akshat/ros2_ws/src/leo_rover/models/ZED2.dae
- link zed2_tilt_head_link: geometry collision mesh filename=/home/akshat/ros2_ws/src/leo_rover/models/Manfrotto_head.dae; visual mesh filename=/home/akshat/ros2_ws/src/leo_rover/models/Manfrotto_head.dae

File: leo_rover/urdf/probe.urdf (robot description, URDF)
Before this commit: robot probe, 1 links, 0 joints
Links:
- link probe_link: geometry collision mesh filename=/home/akshat/ros2_ws/src/leo_rover/models/Probe.dae; visual mesh filename=/home/akshat/ros2_ws/src/leo_rover/models/Probe.dae

File: leo_worlds/worlds/marsyard2022.world.xacro (robot description, xacro)
@@ -30,5 +30,5 @@
     </scene>
     <include>
-      <uri>/home/dillon/myROS2WS/src/leo_worlds/models/marsyard2022_terrain</uri>
+      <uri>/home/akshat/ros2_ws/src/leo_worlds/models/marsyard2022_terrain</uri>
     </include>
     <xacro:include filename="sdf/landmark.sdf.xacro" />

Commit message: new branch

File: leo_rover/urdf/leo_erc_sim.urdf (robot description, URDF)
Before this commit: robot leo_erc_sim, 22 links, 21 joints
Links:
- link base_link: geometry collision mesh filename=/home/aditi/ERC/leo_rover/models/Chassis_outline.stl; visual mesh filename=/home/aditi/ERC/leo_rover/models/Chassis.dae
- link erc_payload_link: geometry collision mesh filename=/home/aditi/ERC/leo_rover/models/ERC2021payload_outline.dae; visual mesh filename=/home/aditi/ERC/leo_rover/models/ERC2021payload.dae
- link rocker_L_link: geometry collision mesh filename=/home/aditi/ERC/leo_rover/models/Rocker_outline.stl; visual mesh filename=/home/aditi/ERC/leo_rover/models/Rocker.dae
- link rocker_R_link: geometry collision mesh filename=/home/aditi/ERC/leo_rover/models/Rocker_outline.stl; visual mesh filename=/home/aditi/ERC/leo_rover/models/Rocker.dae
- link wheel_FL_link: geometry collision cylinder length=0.04 radius=0.0625; collision cylinder length=0.07 radius=0.057
- link wheel_FR_link: geometry collision cylinder length=0.04 radius=0.0625; collision cylinder length=0.07 radius=0.057
- link wheel_RL_link: geometry collision cylinder length=0.04 radius=0.0625; collision cylinder length=0.07 radius=0.057
- link wheel_RR_link: geometry collision cylinder length=0.04 radius=0.0625; collision cylinder length=0.07 radius=0.057
- link zed2_camera_center: geometry collision mesh filename=/home/aditi/ERC/leo_rover/models/ZED2.dae; visual mesh filename=/home/aditi/ERC/leo_rover/models/ZED2.dae
- link zed2_tilt_head_link: geometry collision mesh filename=/home/aditi/ERC/leo_rover/models/Manfrotto_head.dae; visual mesh filename=/home/aditi/ERC/leo_rover/models/Manfrotto_head.dae

File: leo_rover/urdf/probe.urdf (robot description, URDF)
Before this commit: robot probe, 1 links, 0 joints
Links:
- link probe_link: geometry collision mesh filename=/home/aditi/ERC/leo_rover/models/Probe.dae; visual mesh filename=/home/aditi/ERC/leo_rover/models/Probe.dae

Commit message: corrected opencv

File: leo_rover/urdf/leo_erc_sim.urdf (robot description, URDF)
Before this commit: robot leo_erc_sim, 22 links, 21 joints
Links:
- link base_link: geometry collision mesh filename=/home/akshat/ros2_ws/src/leo_rover/models/Chassis_outline.s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; visual mesh filename=/home/akshat/ros2_ws/src/leo_rover/models/Chassis.dae
- link erc_payload_link: geometry collision mesh filename=/home/akshat/ros2_ws/src/leo_rover/models/ERC2021payload_ou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; visual mesh filename=/home/akshat/ros2_ws/src/leo_rover/models/ERC2021payload.dae
- link rocker_L_link: geometry collision mesh filename=/home/akshat/ros2_ws/src/leo_rover/models/Rocker_outline.stl; visual mesh filename=/home/akshat/ros2_ws/src/leo_rover/models/Rocker.dae
- link rocker_R_link: geometry collision mesh filename=/home/akshat/ros2_ws/src/leo_rover/models/Rocker_outline.stl; visual mesh filename=/home/akshat/ros2_ws/src/leo_rover/models/Rocker.dae
- link wheel_FL_link: geometry collision cylinder length=0.04 radius=0.0625; collision cylinder length=0.07 radius=0.057
- link wheel_FR_link: geometry collision cylinder length=0.04 radius=0.0625; collision cylinder length=0.07 radius=0.057
- link wheel_RL_link: geometry collision cylinder length=0.04 radius=0.0625; collision cylinder length=0.07 radius=0.057
- link wheel_RR_link: geometry collision cylinder length=0.04 radius=0.0625; collision cylinder length=0.07 radius=0.057
- link zed2_camera_center: geometry collision mesh filename=/home/akshat/ros2_ws/src/leo_rover/models/ZED2.dae; visual mesh filename=/home/akshat/ros2_ws/src/leo_rover/models/ZED2.dae
- link zed2_tilt_head_link: geometry collision mesh filename=/home/akshat/ros2_ws/src/leo_rover/models/Manfrotto_head.dae; visual mesh filename=/home/akshat/ros2_ws/src/leo_rover/models/Manfrotto_head.dae

File: leo_rover/urdf/probe.urdf (robot description, URDF)
Before this commit: robot probe, 1 links, 0 joints
Links:
- link probe_link: geometry collision mesh filename=/home/akshat/ros2_ws/src/leo_rover/models/Probe.dae; visual mesh filename=/home/akshat/ros2_ws/src/leo_rover/models/Probe.dae
