Commit message: Compltete

File: ros2_ws/src/leo_rover/urdf/leo_erc_sim.urdf (robot description, URDF)
Before this commit: robot leo_erc_sim, 22 links, 21 joints
Links:
- link base_link: geometry collision mesh filename=/home/akshat/myROS2WS/src/leo_rover/models/Chassis_outline.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; visual mesh filename=/home/akshat/myROS2WS/src/leo_rover/models/Chassis.dae
- link erc_payload_link: geometry collision mesh filename=/home/akshat/myROS2WS/src/leo_rover/models/ERC2021payload_o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; visual mesh filename=/home/akshat/myROS2WS/src/leo_rover/models/ERC2021payload.d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
- link rocker_L_link: geometry collision mesh filename=/home/akshat/myROS2WS/src/leo_rover/models/Rocker_outline.s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; visual mesh filename=/home/akshat/myROS2WS/src/leo_rover/models/Rocker.dae
- link rocker_R_link: geometry collision mesh filename=/home/akshat/myROS2WS/src/leo_rover/models/Rocker_outline.s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; visual mesh filename=/home/akshat/myROS2WS/src/leo_rover/models/Rocker.dae
- link wheel_FL_link: geometry collision cylinder length=0.04 radius=0.0625; collision cylinder length=0.07 radius=0.057
- link wheel_FR_link: geometry collision cylinder length=0.04 radius=0.0625; collision cylinder length=0.07 radius=0.057
- link wheel_RL_link: geometry collision cylinder length=0.04 radius=0.0625; collision cylinder length=0.07 radius=0.057
- link wheel_RR_link: geometry collision cylinder length=0.04 radius=0.0625; collision cylinder length=0.07 radius=0.057
- link zed2_camera_center: geometry collision mesh filename=/home/akshat/myROS2WS/src/leo_rover/models/ZED2.dae; visual mesh filename=/home/akshat/myROS2WS/src/leo_rover/models/ZED2.dae
- link zed2_tilt_head_link: geometry collision mesh filename=/home/akshat/myROS2WS/src/leo_rover/models/Manfrotto_head.d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; visual mesh filename=/home/akshat/myROS2WS/src/leo_rover/models/Manfrotto_head.d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

File: ros2_ws/src/leo_rover/urdf/probe.urdf (robot description, URDF)
Before this commit: robot probe, 1 links, 0 joints
Links:
- link probe_link: geometry collision mesh filename=/home/akshat/myROS2WS/src/leo_rover/models/Probe.dae; visual mesh filename=/home/akshat/myROS2WS/src/leo_rover/models/Probe.dae
